File: ESP32-PDM.kicad_sch (KiCad schematic)
At the start: 5 parts, among them J1 Conn_02x04_Top_Bottom, J2 Conn_02x06_Top_Bottom

Commit message: PCB first version
Parts:
- added H2: MountingHole, MountingHole:MountingHole_3mm, symbol Mechanical:MountingHole
- J1: value Conn_02x04_Top_Bottom -> 5569-08A2-210
Changed lines of the file:
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@@
 	(label "OUT4"
 		(at 54.61 104.14 0)
-		(fields_autoplaced yes)
 		(effects
 			(font
@@
 	(label "DIAG2"
 		(at 102.87 116.84 0)
-		(fields_autoplaced yes)
 		(effects
 			(font
@@
 	(label "IN4"
 		(at 124.46 109.22 0)
-		(fields_autoplaced yes)
 		(effects
 			(font
@@
 	(label "DIAG3"
 		(at 54.61 90.17 0)
-		(fields_autoplaced yes)
 		(effects
 			(font
@@
 	(label "IN1"
 		(at 102.87 109.22 0)
-		(fields_autoplaced yes)
 		(effects
 			(font
@@
 	(label "IN2"
 		(at 102.87 114.3 0)
-		(fields_autoplaced yes)
 		(effects
 			(font
@@
 	(label "IN1"
 		(at 31.75 50.8 0)
-		(fields_autoplaced yes)
 		(effects
 			(font
@@
 	(label "DIAG2"
 		(at 54.61 72.39 0)
-		(fields_autoplaced yes)
 		(effects
 			(font
@@
 	(label "OUT4"
 		(at 120.65 77.47 0)
-		(fields_autoplaced yes)
 		(effects
 			(font
@@
 	(label "DIAG1"
 		(at 54.61 54.61 0)
-		(fields_autoplaced yes)
 		(effects
 			(font
@@
 	(label "IN4"
 		(at 31.75 104.14 0)
-		(fields_autoplaced yes)
 		(effects
 			(font
@@
 	(label "DIAG4"
 		(at 54.61 107.95 0)
-		(fields_autoplaced yes)
 		(effects
 			(font
@@
 	(label "IN3"
 		(at 31.75 86.36 0)
-		(fields_autoplaced yes)
 		(effects
 			(font
@@
 	(label "OUT1"
 		(at 54.61 50.8 0)
-		(fields_autoplaced yes)
 		(effects
 			(font
@@
 	(label "DIAG3"
 		(at 102.87 121.92 0)
-		(fields_autoplaced yes)
 		(effects
 			(font
@@
 	(label "OUT2"
 		(at 120.65 82.55 0)
-		(fields_autoplaced yes)
 		(effects
 			(font
@@
 	(label "OUT3"
 		(at 120.65 80.01 0)
-		(fields_autoplaced yes)
 		(effects
 			(font
@@
 	(label "DIAG4"
 		(at 124.46 111.76 0)
-		(fields_autoplaced yes)
 		(effects
 			(font
@@
 	(label "IN3"
 		(at 102.87 119.38 0)
-		(fields_autoplaced yes)
 		(effects
 			(font
@@
 	(label "IN2"
 		(at 31.75 68.58 0)
-		(fields_autoplaced yes)
 		(effects
 			(font
@@
 	(label "OUT2"
 		(at 54.61 68.58 0)
-		(fields_autoplaced yes)
 		(effects
 			(font
@@
 	(label "DIAG1"
 		(at 102.87 111.76 0)
-		(fields_autoplaced yes)
 		(effects
 			(font
@@
 	(label "OUT1"
 		(at 120.65 85.09 0)
-		(fields_autoplaced yes)
 		(effects
 			(font
@@
 	(label "OUT3"
 		(at 54.61 86.36 0)
-		(fields_autoplaced yes)
 		(effects
 			(font
@@
 			)
 		)
-		(property "Value" "Conn_02x04_Top_Bottom"
+		(property "Value" "5569-08A2-210"
 			(at 114.3 73.66 0)
 			(effects
@@
 					(unit 1)
 				)
+			)
+		)
+	)
+	(symbol
+		(lib_id "Mechanical:MountingHole")
+		(at 39.37 148.59 0)
+		(unit 1)
+		(exclude_from_sim yes)
+		(in_bom no)
+		(on_board yes)
+		(dnp no)
+		(fields_autoplaced yes)
+		(property "Reference" "H2"
+			(at 41.91 147.3199 0)
+			(effects
+				(font
+					(size 1.27 1.27)
+				)
+				(justify left)
+			)
+		)
+		(property "Value" "MountingHole"
+			(at 41.91 149.8599 0)
+			(effects
+				(font
+					(size 1.27 1.27)
+				)
+				(justify left)
+			)
+		)
+		(property "Footprint" "MountingHole:MountingHole_3mm"
+			(at 39.37 148.59 0)
+			(effects
+				(font
+					(size 1.27 1.27)
+				)
+				(hide yes)
+			)
+		)
+		(property "Datasheet" "~"
+			(at 39.37 148.59 0)
+			(effects
+				(font
+					(size 1.27 1.27)
+				)
+				(hide yes)
+			)
+		)
+		(property "Description" "Mounting Hole without connection"
+			(at 39.37 148.59 0)
+			(effects
+				(font
+					(size 1.27 1.27)
+				)
+				(hide yes)
+			)
+		)
+		(instances
+			(project "ESP32-PDM"
+				(path "/77f0f044-4c8a-4320-9763-77a575781bec"
+					(reference "H2")
+					(unit 1)
+				)
